Commit message: Build initial E5 mechArm Gazebo simulation

File: E5_fixed_pick_place/ros2_ws/src/e5_arm_sim/urdf/mecharm_270_m5_sim.urdf.xacro (robot description, xacro)
@@ -2,4 +2,11 @@
 <robot xmlns:ns0="http://www.ros.org/wiki/xacro" name="firefighter">
   <ns0:property name="width" value=".2" />
+  <!-- Fix the robot base to the simulation world -->
+  <link name="world"/>
+  <joint name="world_to_base" type="fixed">
+    <parent link="world"/>
+    <child link="base"/>
+    <origin xyz="0 0 0.42" rpy="0 0 0"/>
+  </joint>
   <link name="base">
     <inertial>
@@ -10,5 +17,5 @@
     <visual>
       <geometry>
-        <mesh filename="package://mycobot_description/urdf/mecharm_270_m5/base.dae" />
+        <mesh filename="file://$(find mycobot_description)/urdf/mecharm_270_m5/base.dae" />
       </geometry>
       <origin xyz=" 0 0 0 " rpy=" 0 0 -3.1415926" />
@@ -16,5 +23,5 @@
     <collision>
       <geometry>
-        <mesh filename="package://mycobot_description/urdf/mecharm_270_m5/base.dae" />
+        <mesh filename="file://$(find mycobot_description)/urdf/mecharm_270_m5/base.dae" />
       </geometry>
       <origin xyz=" 0 0 0 " rpy=" 0 0 -3.1415926" />
@@ -29,5 +36,5 @@
     <visual>
       <geometry>
-        <mesh filename="package://mycobot_description/urdf/mecharm_270_m5/link1.dae" />
+        <mesh filename="file://$(find mycobot_description)/urdf/mecharm_270_m5/link1.dae" />
       </geometry>
       <origin xyz="0 0 -0.132 " rpy=" 0 0 0" />
@@ -35,5 +42,5 @@
     <collision>
       <geometry>
-        <mesh filename="package://mycobot_description/urdf/mecharm_270_m5/link1.dae" />
+        <mesh filename="file://$(find mycobot_description)/urdf/mecharm_270_m5/link1.dae" />
       </geometry>
       <origin xyz="0 0 -0.132 " rpy=" 0 0 0" />
@@ -48,5 +55,5 @@
     <visual>
       <geometry>
-        <mesh filename="package://mycobot_description/urdf/mecharm_270_m5/link2.dae" />
+        <mesh filename="file://$(find mycobot_description)/urdf/mecharm_270_m5/link2.dae" />
       </geometry>
       <origin xyz="-0.005 0.21 0.002  " rpy=" 1.5708 -3.1415926 0" />
@@ -54,5 +61,5 @@
     <collision>
       <geometry>
-        <mesh filename="package://mycobot_description/urdf/mecharm_270_m5/link2.dae" />
+        <mesh filename="file://$(find mycobot_description)/urdf/mecharm_270_m5/link2.dae" />
       </geometry>
       <origin xyz="-0.005  -0.21 0.002  " rpy=" 1.5708 -3.1415926 0" />
@@ -67,5 +74,5 @@
     <visual>
       <geometry>
-        <mesh filename="package://mycobot_description/urdf/mecharm_270_m5/link3.dae" />
+        <mesh filename="file://$(find mycobot_description)/urdf/mecharm_270_m5/link3.dae" />
       </geometry>
       <origin xyz="-0.09 0.306 0.005 " rpy="1.5708 3.1415926  0" />
@@ -73,5 +80,5 @@
     <collision>
       <geometry>
-        <mesh filename="package://mycobot_description/urdf/mecharm_270_m5/link3.dae" />
+        <mesh filename="file://$(find mycobot_description)/urdf/mecharm_270_m5/link3.dae" />
       </geometry>
       <origin xyz="-0.09 0.306 0.005" rpy="1.5708 3.1415926 0" />
@@ -86,5 +93,5 @@
     <visual>
       <geometry>
-        <mesh filename="package://mycobot_description/urdf/mecharm_270_m5/link4.dae" />
+        <mesh filename="file://$(find mycobot_description)/urdf/mecharm_270_m5/link4.dae" />
       </geometry>
       <origin xyz="0.009 -0.311 -0.228" rpy=" 0 1.5708 1.5708" />
@@ -92,5 +99,5 @@
     <collision>
       <geometry>
-        <mesh filename="package://mycobot_description/urdf/mecharm_270_m5/link4.dae" />
+        <mesh filename="file://$(find mycobot_description)/urdf/mecharm_270_m5/link4.dae" />
       </geometry>
       <origin xyz="0.009 -0.311  -0.228" rpy=" 0 1.5708  1.5708" />
@@ -105,5 +112,5 @@
     <visual>
       <geometry>
-        <mesh filename="package://mycobot_description/urdf/mecharm_270_m5/link5.dae" />
+        <mesh filename="file://$(find mycobot_description)/urdf/mecharm_270_m5/link5.dae" />
       </geometry>
       <origin xyz="-0.292 -0.318 -0.007" rpy=" 1.5708 0 3.1415926" />
@@ -111,5 +118,5 @@
     <collision>
       <geometry>
-        <mesh filename="package://mycobot_description/urdf/mecharm_270_m5/link5.dae" />
+        <mesh filename="file://$(find mycobot_description)/urdf/mecharm_270_m5/link5.dae" />
       </geometry>
       <origin xyz="-0.292 -0.318 -0.007 " rpy=" 1.5708 0 3.1415926" />
@@ -124,5 +131,5 @@
     <visual>
       <geometry>
-        <mesh filename="package://mycobot_description/urdf/mecharm_270_m5/link6.dae" />
+        <mesh filename="file://$(find mycobot_description)/urdf/mecharm_270_m5/link6.dae" />
       </geometry>
       <origin xyz="-0.1645 0.0536 -0.211 " rpy=" 0 1.5708 0" />
@@ -130,5 +137,5 @@
     <collision>
       <geometry>
-        <mesh filename="package://mycobot_description/urdf/mecharm_270_m5/link6.dae" />
+        <mesh filename="file://$(find mycobot_description)/urdf/mecharm_270_m5/link6.dae" />
       </geometry>
       <origin xyz="-0.1645 0.0536 -0.211 " rpy=" 0 1.5708 0" />
@@ -143,5 +150,5 @@
     <visual>
       <geometry>
-        <mesh filename="package://mycobot_description/urdf/adaptive_gripper/gripper_base.dae" />
+        <mesh filename="file://$(find mycobot_description)/urdf/adaptive_gripper/gripper_base.dae" />
       </geometry>
       <origin xyz="0.0 0 -0.012 " rpy=" 0 0 0" />
@@ -149,5 +156,5 @@
     <collision>
       <geometry>
-        <mesh filename="package://mycobot_description/urdf/adaptive_gripper/gripper_base.dae" />
+        <mesh filename="file://$(find mycobot_description)/urdf/adaptive_gripper/gripper_base.dae" />
       </geometry>
       <origin xyz="0.0 0 -0.012 " rpy=" 0 0 0" />
@@ -162,5 +169,5 @@
     <visual>
       <geometry>
-        <mesh filename="package://mycobot_description/urdf/adaptive_gripper/gripper_left1.dae" />
+        <mesh filename="file://$(find mycobot_description)/urdf/adaptive_gripper/gripper_left1.dae" />
       </geometry>
       <origin xyz="0.039 -0.0133 -0.012 " rpy=" 0 0 0" />
@@ -168,5 +175,5 @@
     <collision>
       <geometry>
-        <mesh filename="package://mycobot_description/urdf/adaptive_gripper/gripper_left1.dae" />
+        <mesh filename="file://$(find mycobot_description)/urdf/adaptive_gripper/gripper_left1.dae" />
       </geometry>
       <origin xyz="0.039 -0.0133 -0.012 " rpy=" 0 0 0" />
@@ -181,5 +188,5 @@
     <visual>
       <geometry>
-        <mesh filename="package://mycobot_description/urdf/adaptive_gripper/gripper_left2.dae" />
+        <mesh filename="file://$(find mycobot_description)/urdf/adaptive_gripper/gripper_left2.dae" />
       </geometry>
       <origin xyz="0.005 -0.0195 -0.012 " rpy=" 0 0 0" />
@@ -187,5 +194,5 @@
     <collision>
       <geometry>
-        <mesh filename="package://mycobot_description/urdf/adaptive_gripper/gripper_left2.dae" />
+        <mesh filename="file://$(find mycobot_description)/urdf/adaptive_gripper/gripper_left2.dae" />
       </geometry>
       <origin xyz="0.005 -0.0195 -0.012 " rpy=" 0 0 0" />
@@ -200,5 +207,5 @@
     <visual>
       <geometry>
-        <mesh filename="package://mycobot_description/urdf/adaptive_gripper/gripper_left3.dae" />
+        <mesh filename="file://$(find mycobot_description)/urdf/adaptive_gripper/gripper_left3.dae" />
       </geometry>
       <origin xyz="0.012 0.0025 -0.012 " rpy=" 0 0 0" />
@@ -206,5 +213,5 @@
     <collision>
       <geometry>
-        <mesh filename="package://mycobot_description/urdf/adaptive_gripper/gripper_left3.dae" />
+        <mesh filename="file://$(find mycobot_description)/urdf/adaptive_gripper/gripper_left3.dae" />
       </geometry>
       <origin xyz="0.012 0.0025 -0.012 " rpy=" 0 0 0" />
@@ -219,5 +226,5 @@
     <visual>
       <geometry>
-        <mesh filename="package://mycobot_description/urdf/adaptive_gripper/gripper_right1.dae" />
+        <mesh filename="file://$(find mycobot_description)/urdf/adaptive_gripper/gripper_right1.dae" />
       </geometry>
       <origin xyz="-0.039 -0.0133 -0.012 " rpy=" 0 0 0" />
@@ -225,5 +232,5 @@
     <collision>
       <geometry>
-        <mesh filename="package://mycobot_description/urdf/adaptive_gripper/gripper_right1.dae" />
+        <mesh filename="file://$(find mycobot_description)/urdf/adaptive_gripper/gripper_right1.dae" />
       </geometry>
       <origin xyz="-0.039 -0.0133 -0.012 " rpy=" 0 0 0" />
@@ -238,5 +245,5 @@
     <visual>
       <geometry>
-        <mesh filename="package://mycobot_description/urdf/adaptive_gripper/gripper_right2.dae" />
+        <mesh filename="file://$(find mycobot_description)/urdf/adaptive_gripper/gripper_right2.dae" />
       </geometry>
       <origin xyz="-0.005 -0.0195 -0.012 " rpy=" 0 0 0" />
@@ -244,5 +251,5 @@
     <collision>
       <geometry>
-        <mesh filename="package://mycobot_description/urdf/adaptive_gripper/gripper_right2.dae" />
+        <mesh filename="file://$(find mycobot_description)/urdf/adaptive_gripper/gripper_right2.dae" />
       </geometry>
       <origin xyz="-0.005 -0.0195 -0.012 " rpy=" 0 0 0" />
@@ -257,5 +264,5 @@
     <visual>
       <geometry>
-        <mesh filename="package://mycobot_description/urdf/adaptive_gripper/gripper_right3.dae" />
+        <mesh filename="file://$(find mycobot_description)/urdf/adaptive_gripper/gripper_right3.dae" />
       </geometry>
       <origin xyz="-0.012 0.0025 -0.012 " rpy=" 0 0 0" />
@@ -263,5 +270,5 @@
     <collision>
       <geometry>
-        <mesh filename="package://mycobot_description/urdf/adaptive_gripper/gripper_right3.dae" />
+        <mesh filename="file://$(find mycobot_description)/urdf/adaptive_gripper/gripper_right3.dae" />
       </geometry>
       <origin xyz="-0.012 0.0025 -0.012" rpy=" 0 0 0" />
@@ -362,3 +369,87 @@
     <mimic joint="gripper_controller" multiplier="1.0" offset="0" />
   </joint>
+  <!-- Gazebo ros2_control hardware interfaces -->
+  <ros2_control name="GazeboSystem" type="system">
+    <hardware>
+      <plugin>gazebo_ros2_control/GazeboSystem</plugin>
+    </hardware>
+    <joint name="joint1_to_base">
+      <command_interface name="position"/>
+      <state_interface name="position"/>
+      <state_interface name="velocity"/>
+    </joint>
+    <joint name="joint2_to_joint1">
+      <command_interface name="position"/>
+      <state_interface name="position"/>
+      <state_interface name="velocity"/>
+    </joint>
+    <joint name="joint3_to_joint2">
+      <command_interface name="position"/>
+      <state_interface name="position"/>
+      <state_interface name="velocity"/>
+    </joint>
+    <joint name="joint4_to_joint3">
+      <command_interface name="position"/>
+      <state_interface name="position"/>
+      <state_interface name="velocity"/>
+    </joint>
+    <joint name="joint5_to_joint4">
+      <command_interface name="position"/>
+      <state_interface name="position"/>
+      <state_interface name="velocity"/>
+    </joint>
+    <joint name="joint6_to_joint5">
+      <command_interface name="position"/>
+      <state_interface name="position"/>
+      <state_interface name="velocity"/>
+    </joint>
+    <joint name="gripper_controller">
+      <command_interface name="position"/>
+      <state_interface name="position"/>
+      <state_interface name="velocity"/>
+    </joint>
+    <joint name="gripper_base_to_gripper_left2">
+      <param name="mimic">gripper_controller</param>
+      <param name="multiplier">1.0</param>
+      <command_interface name="position"/>
+      <state_interface name="position"/>
+      <state_interface name="velocity"/>
+    </joint>
+    <joint name="gripper_left3_to_gripper_left1">
+      <param name="mimic">gripper_controller</param>
+      <param name="multiplier">-1.0</param>
+      <command_interface name="position"/>
+      <state_interface name="position"/>
+      <state_interface name="velocity"/>
+    </joint>
+    <joint name="gripper_base_to_gripper_right3">
+      <param name="mimic">gripper_controller</param>
+      <param name="multiplier">-1.0</param>
+      <command_interface name="position"/>
+      <state_interface name="position"/>
+      <state_interface name="velocity"/>
+    </joint>
+    <joint name="gripper_base_to_gripper_right2">
+      <param name="mimic">gripper_controller</param>
+      <param name="multiplier">-1.0</param>
+      <command_interface name="position"/>
+      <state_interface name="position"/>
+      <state_interface name="velocity"/>
+    </joint>
+    <joint name="gripper_right3_to_gripper_right1">
+      <param name="mimic">gripper_controller</param>
+      <param name="multiplier">1.0</param>
+      <command_interface name="position"/>
+      <state_interface name="position"/>
+      <state_interface name="velocity"/>
+    </joint>
+  </ros2_control>
+  <!-- Load ros2_control inside Gazebo Classic -->
+  <gazebo>
+    <plugin
+      name="gazebo_ros2_control"
+      filename="libgazebo_ros2_control.so">
+      <parameters>$(find e5_arm_sim)/config/controllers.yaml</parameters>
+    </plugin>
+  </gazebo>
 </robot>

Commit message: fix(E5): improve Gazebo grasp simulation

File: E5_fixed_pick_place/ros2_ws/src/e5_arm_sim/urdf/mecharm_270_m5_sim.urdf.xacro (robot description, xacro)
@@ -1,5 +1,5 @@
 <?xml version='1.0' encoding='utf-8'?>
-<robot xmlns:ns0="http://www.ros.org/wiki/xacro" name="firefighter">
-  <ns0:property name="width" value=".2" />
+<robot xmlns:xacro="http://www.ros.org/wiki/xacro" name="firefighter">
+  <xacro:property name="width" value=".2" />
   <!-- Fix the robot base to the simulation world -->
   <link name="world"/>
@@ -370,4 +370,28 @@
   </joint>
   <!-- Gazebo ros2_control hardware interfaces -->
+  <!-- Virtual frame at the centre between the gripper fingers -->
+  <link name="grasp_point"/>
+  <joint name="gripper_base_to_grasp_point" type="fixed">
+    <parent link="gripper_base"/>
+    <child link="grasp_point"/>
+    <origin xyz="0 0.060 0" rpy="0 0 0"/>
+  </joint>
+  <!-- e5_high_friction - improve simulated grasping -->
+  <gazebo reference="gripper_left1">
+    <mu1>10.0</mu1>
+    <mu2>10.0</mu2>
+    <kp>1000000.0</kp>
+    <kd>10.0</kd>
+    <minDepth>0.001</minDepth>
+    <maxVel>0.1</maxVel>
+  </gazebo>
+  <gazebo reference="gripper_right1">
+    <mu1>10.0</mu1>
+    <mu2>10.0</mu2>
+    <kp>1000000.0</kp>
+    <kd>10.0</kd>
+    <minDepth>0.001</minDepth>
+    <maxVel>0.1</maxVel>
+  </gazebo>
   <ros2_control name="GazeboSystem" type="system">
     <hardware>

Commit message: feat(E5): automate Gazebo pick and place

File: E5_fixed_pick_place/ros2_ws/src/e5_arm_sim/urdf/mecharm_270_m5_sim.urdf.xacro (robot description, xacro)
@@ -173,9 +173,9 @@
       <origin xyz="0.039 -0.0133 -0.012 " rpy=" 0 0 0" />
     </visual>
-    <collision>
-      <geometry>
-        <mesh filename="file://$(find mycobot_description)/urdf/adaptive_gripper/gripper_left1.dae" />
-      </geometry>
-      <origin xyz="0.039 -0.0133 -0.012 " rpy=" 0 0 0" />
+    <collision name="left_finger_box">
+      <origin xyz="0.0369 -0.0104 -0.007" rpy="0 0 0"/>
+      <geometry>
+        <box size="0.050 0.015 0.014"/>
+      </geometry>
     </collision>
   </link>
@@ -230,9 +230,9 @@
       <origin xyz="-0.039 -0.0133 -0.012 " rpy=" 0 0 0" />
     </visual>
-    <collision>
-      <geometry>
-        <mesh filename="file://$(find mycobot_description)/urdf/adaptive_gripper/gripper_right1.dae" />
-      </geometry>
-      <origin xyz="-0.039 -0.0133 -0.012 " rpy=" 0 0 0" />
+    <collision name="right_finger_box">
+      <origin xyz="-0.0369 -0.0104 -0.007" rpy="0 0 0"/>
+      <geometry>
+        <box size="0.050 0.015 0.014"/>
+      </geometry>
     </collision>
   </link>
@@ -370,4 +370,23 @@
   </joint>
   <!-- Gazebo ros2_control hardware interfaces -->
+  <!-- Preserved attachment frame for the pick object -->
+  <link name="grasp_attach_link">
+    <inertial>
+      <mass value="0.001"/>
+      <inertia
+        ixx="0.000001" ixy="0.0" ixz="0.0"
+        iyy="0.000001" iyz="0.0" izz="0.000001"/>
+    </inertial>
+  </link>
+  <joint name="link6_to_grasp_attach_link" type="fixed">
+    <parent link="link6"/>
+    <child link="grasp_attach_link"/>
+    <origin
+      xyz="-0.000627 0.004725 0.121851"
+      rpy="-3.1415 0.00014 -1.5691"/>
+  </joint>
+  <gazebo reference="link6_to_grasp_attach_link">
+    <preserveFixedJoint>true</preserveFixedJoint>
+  </gazebo>
   <!-- Virtual frame at the centre between the gripper fingers -->
   <link name="grasp_point"/>
